File: ssmm.kicad_sch (KiCad schematic)
At the start: 20 parts, among them J1 Accelerometer_IN, J4 Accelerometer_AUX, SW1 SW_Push, U1 ESP-12E, U2 AMS1117-3.3

Commit message: Usability++
Parts:
- R1: value 4.7k -> 10K
- R4, R5: value 180k -> 100K
Changed lines of the file:
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@@
 			)
 		)
-		(property "Value" "4.7k"
+		(property "Value" "10K"
 			(at 98.0186 78.613 0)
 			(effects
@@
 			)
 		)
-		(property "Value" "180k"
+		(property "Value" "100K"
 			(at 99.2886 104.013 0)
 			(effects
@@
 			)
 		)
-		(property "Value" "180k"
+		(property "Value" "100K"
 			(at 90.297 96.7486 0)
 			(effects
